File: tx.sch (KiCad schematic (older format))
At the start: 37 parts, among them T2 Transformer_1P_SS, U10 TLV2464CD, U11 SN74CBT3253

Commit message: A lot of minor layout changes
Connections:
- net at R21.1: now also T2.5 (SB); no longer T2.3 (SA)
- net at R23.1: now also T2.3 (SA); no longer T2.5 (SB)
Changed lines of the file:
@@
 EESchema Schematic File Version 4
-EELAYER 30 0
+LIBS:DeltaSDR-cache
+EELAYER 29 0
 EELAYER END
 $Descr A4 11693 8268
@@
 $EndComp
 Wire Wire Line
-	5725 3100 5575 3100
-Wire Wire Line
-	5575 3100 5575 3250
-Wire Wire Line
 	5575 3250 5475 3250
-Wire Wire Line
-	5725 3500 5575 3500
-Wire Wire Line
-	5575 3500 5575 3350
-Wire Wire Line
-	5575 3350 5475 3350
 Wire Wire Line
 	5725 3300 5675 3300
@@
 Wire Wire Line
 	4825 2000 5025 2000
+Wire Wire Line
+	5650 3350 5650 3100
+Wire Wire Line
+	5650 3100 5725 3100
+Wire Wire Line
+	5475 3350 5650 3350
+Wire Wire Line
+	5575 3250 5575 3500
+Wire Wire Line
+	5575 3500 5725 3500
 $EndSCHEMATC
